File: pcb/mainboard/audio.kicad_sch (KiCad schematic)
At the start: 32 parts, among them J701 Conn_01x02, J702 Conn_01x02, J703 AudioJack3_SwitchT, U701 WM8960

Commit message: - pcb: migrate to latest kicad, r0p1
Parts:
- J703: footprint footprints:Jack_3.5mm_PJ327E_5A -> footprints:PJ-327E
Connections:
- net +3.3VA is gone; now on net +3V3: R708.1
Changed lines of the file:
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@@
   (title_block
     (title "Archer Mainboard")
-    (date "2021-05-06")
-    (rev "R0.1 draft")
+    (date "2021-05-13")
+    (rev "R0.1")
     (company "Copyright EI-2030 2021. / Engineer: Wenting Zhang")
     (comment 2 "MERCHANTABILITY, SATISFACTORY QUALITY AND FITNESS FOR A PARTICULAR PURPOSE.")
@@
     (pin "1")
   )
-  (symbol (lib_id "power:+3.3VA") (at 204.47 66.04 0) (unit 1)
-    (in_bom yes) (on_board yes)
-    (property "Reference" "#PWR0714" (id 0) (at 204.47 69.85 0)
-      (effects (font (size 1.27 1.27)) hide)
-    )
-    (property "Value" "+3.3VA" (id 1) (at 205.74 62.23 0))
+  (symbol (lib_id "power:+3V3") (at 204.47 66.04 0) (unit 1)
+    (in_bom yes) (on_board yes)
+    (property "Reference" "#PWR0169" (id 0) (at 204.47 69.85 0)
+      (effects (font (size 1.27 1.27)) hide)
+    )
+    (property "Value" "+3V3" (id 1) (at 201.93 62.23 0))
     (property "Footprint" "" (id 2) (at 204.47 66.04 0)
       (effects (font (size 1.27 1.27)) hide)
@@
       (effects (font (size 1.27 1.27)) (justify right))
     )
-    (property "Footprint" "footprints:Jack_3.5mm_PJ327E_5A" (id 2) (at 212.09 106.68 0)
-      (effects (font (size 1.27 1.27)) hide)
-    )
+    (property "Footprint" "footprints:PJ-327E" (id 2) (at 212.09 106.68 0)
+      (effects (font (size 1.27 1.27)) hide)
+    )
