File: pcb/mainboard/cpu.kicad_sch (KiCad schematic)
At the start: 0 parts

Commit message: - pcb: switch to imx7 for the prototype
Parts:
- added C? (x16): 220nF, Capacitor_SMD:C_0402_1005Metric, symbol Device:C
- added C? (x2): DNP/18pF, Capacitor_SMD:C_0402_1005Metric, symbol Device:C
- added C? (x6): 2.2uF, Capacitor_SMD:C_0402_1005Metric, symbol Device:C
- added C? (x2): 18pF, Capacitor_SMD:C_0402_1005Metric, symbol Device:C
- added L?: 120R, Inductor_SMD:L_0603_1608Metric, symbol Device:L
- added R? (x2): 200/1%, Resistor_SMD:R_0603_1608Metric, symbol Device:R
- added R? (x6): 10K, Resistor_SMD:R_0603_1608Metric, symbol Device:R
- added R? (x2): DNP/10K, Resistor_SMD:R_0603_1608Metric, symbol Device:R
- added R?: 100K/1%, Resistor_SMD:R_0603_1608Metric, symbol Device:R
- added R?: 1M, Resistor_SMD:R_0603_1608Metric, symbol Device:R
- added R?: DNP/4.75M, Resistor_SMD:R_0603_1608Metric, symbol Device:R
- added RN? (x3): 10K, Resistor_SMD:R_Array_Convex_4x0402, symbol Device:R_Pack04
- added U? (x10): MCIMX7S5EVM08SC, footprints:BGA-541_25x25_19.0x19.0mm, symbol symbols:MCIMX7S5EVM08SC
- added Y?: 24MHz, Oscillator:Oscillator_SMD_Abracon_ASE-4Pin_3.2x2.5mm, symbol Device:Crystal_GND24
- added Y?: 32.768kHz, Crystal:Crystal_SMD_TXC_9HT11-2Pin_2.0x1.2mm_HandSoldering, symbol Device:Crystal
Connections:
- new net: C?.1, C?.1, L?.2, U?.AB3 (VDDA_ADC2_1P8), U?.AC3 (VDDA_ADC1_1P8), U?.AC4 (VDD_TEMPSENSOR_1P8)
- new net: R?.2, U?.AE4 (TEMPSENSOR_REXT)
- new net: R?.1, U?.A11 (USB_OTG2_REXT)
- new net: C?.1, R?.2, U?.V2 (XTALO), Y?.1
- new net: C?.1, R?.1, U?.V1 (XTALI), Y?.3
- new net: C?.1, R?.2, U?.AD6 (RTC_XTALO), Y?.1
- new net: R?.1, U?.B11 (USB_OTG2_ID)
- new net: R?.1, R?.2, U?.P5 (BOOT_MODE1)
- new net: R?.1, U?.B7 (USB_OTG1_ID)
- new net: C?.1, R?.1, U?.AE6 (RTC_XTALI), Y?.2
- new net: R?.1, R?.2, U?.P4 (BOOT_MODE0)
- new net: C?.1, U?.N17 (PVCC_EPDC_LCD_CAP)
- new net: C?.1, C?.1, U?.J11 (VDD_USB_OTG2_1P0_CAP)
- new net: R?.1, U?.A7 (USB1_OTG1_REXT)
- new net: C?.1, U?.R9 (PVCC_I2C_SPI_UART_CAP)
- new net: C?.1, C?.1, U?.H10 (VDD_USB_OTG1_1P0_CAP)
- new net: C?.1, U?.J9 (PVCC_SAI_SD_CAP)
- new net +1V8: C?.1, C?.1, C?.1, C?.1, C?.1, L?.1, U?.F12 (NVCC_SAI), U?.K18 (NVCC_LCD), U?.L17 (NVCC_EPDC2), U?.M18 (NVCC_EPDC1)
- new net +1V8A: C?.1, U?.V5 (VDD_XTAL_1P8)
- new net +3V3: C?.1, C?.1, C?.1, C?.1, C?.1, C?.1, R?.1, R?.1, RN?.5 (R4.2), RN?.6 (R3.2), RN?.7 (R2.2), RN?.8 (R1.2), U?.F10 (VDD_USB_OTG1_3P3_IN), U?.F9 (VDD_USB_OTG2_3P3_IN), U?.H8 (NVCC_SD2), U?.K8 (NVCC_SD3), U?.L9 (NVCC_SPI), U?.M8 (NVCC_I2C), U?.N9 (NVCC_UART)
- new net +RTC: R?.2, R?.2
- new net +VCCIO_WL: C?.1, U?.E7 (NVCC_SD1)
- new net ADC1_IN0: U?.AD1 (ADC1_IN0)
- new net ADC1_IN1: U?.AD3 (ADC1_IN1)
- new net AP_WAKE_BT: U?.T1 (GPIO_IO11)
- new net BAT_LOW: U?.Y3 (SNVS_TAMPER9)
- new net BT_CFG_1: RN?.4 (R4.1), U?.A22 (LCD1_DATA1)
- new net BT_CFG_10: RN?.5 (R4.2), U?.B24 (LCD1_DATA10)
- new net BT_CFG_11: RN?.8 (R1.2), U?.G20 (LCD1_DATA11)
- new net BT_CFG_12: RN?.2 (R2.1), U?.F21 (LCD1_DATA12)
- new net BT_CFG_13: RN?.7 (R2.2), U?.E22 (LCD1_DATA13)
- new net BT_CFG_14: RN?.6 (R3.2), U?.D23 (LCD1_DATA14)
- new net BT_CFG_2: RN?.5 (R4.2), U?.B22 (LCD1_DATA2)
- new net BT_CFG_3: RN?.6 (R3.2), U?.A23 (LCD1_DATA3)
- new net BT_CFG_4: RN?.3 (R3.1), U?.C22 (LCD1_DATA4)
- new net BT_CFG_5: RN?.8 (R1.2), U?.B23 (LCD1_DATA5)
- new net BT_CFG_6: RN?.7 (R2.2), U?.A24 (LCD1_DATA6)
- new net BT_RST_N: U?.T3 (GPIO_IO13)
- new net BT_WAKE_AP: U?.T2 (GPIO_IO12)
- new net CCM_CLKO2: U?.C4 (SD1_WP)
- new net EXT_PWR_GOOD: U?.AB6 (SNVS_TAMPER2)
- new net GND: C?.2, C?.2, C?.2, C?.2, C?.2, C?.2, C?.2, C?.2, C?.2, C?.2, C?.2, C?.2, C?.2, C?.2, C?.2, C?.2, C?.2, C?.2, C?.2, C?.2, C?.2, C?.2, C?.2, C?.2, C?.2, C?.2, R?.1, R?.1, R?.1, R?.2, R?.2, R?.2, R?.2, RN?.1 (R1.1), RN?.1 (R1.1), RN?.2 (R2.1), RN?.2 (R2.1), RN?.3 (R3.1), RN?.3 (R3.1), RN?.4 (R4.1), RN?.4 (R4.1), U?.AA13 (PCIE_REXT), U?.AB1 (ADC2_IN2), U?.AB2 (ADC2_IN3), U?.AC1 (ADC2_IN0), U?.AC2 (ADC2_IN1), U?.H16 (NVCC_ENET1), U?.P6 (TEST_MODE), U?.U1 (JTAG_MOD), U?.W3 (CCM_CLK2), Y?.2, Y?.4
- new net I2C1_SCL: R?.2, U?.J2 (I2C1_SCL)
- new net I2C1_SDA: R?.2, U?.K1 (I2C1_SDA)
- new net LCD1_CLK: U?.E20 (LCD1_CLK)
- new net LCD1_DE: U?.F25 (LCD1_ENABLE)
- new net LCD1_HSYNC: U?.E25 (LCD1_HSYNC)
- new net LCD1_RESET: U?.C21 (LCD1_RESET)
- new net LCD1_VSYNC: U?.F24 (LCD1_VSYNC)
- new net LCD_D0: U?.D21 (LCD1_DATA0)
- new net LCD_D15: U?.C24 (LCD1_DATA15)
- new net LCD_D16: U?.B25 (LCD1_DATA16)
- new net LCD_D17: U?.G21 (LCD1_DATA17)
- new net LCD_D18: U?.E23 (LCD1_DATA18)
- new net LCD_D19: U?.D24 (LCD1_DATA19)
- new net LCD_D20: U?.C25 (LCD1_DATA20)
- new net LCD_D21: U?.E24 (LCD1_DATA21)
- new net LCD_D22: U?.D25 (LCD1_DATA22)
- new net LCD_D23: U?.G23 (LCD1_DATA23)
- new net LCD_D7: U?.F20 (LCD1_DATA7)
- new net LCD_D8: U?.E21 (LCD1_DATA8)
- new net LCD_D9: U?.C23 (LCD1_DATA9)
- new net MPU_JTAG_TCK: U?.U5 (JTAG_TCK)
- new net MPU_JTAG_TDI: U?.U3 (JTAG_TDI)
- new net MPU_JTAG_TDO: U?.U6 (JTAG_TDO)
- new net MPU_JTAG_TMS: U?.U4 (JTAG_TMS)
- new net MPU_JTAG_TRST: U?.U2 (~JTAG_TRST)
- new net PB_STAT: U?.AC8 (ONOFF)
- new net PMIC_ON_REQ: U?.AB8 (SNVS_PMIC_ON_REQ)
- new net PMIC_STBY_REQ: U?.AC7 (PMIC_STBY_REQ)
- new net POR: U?.R6 (~POR)
- new net SAI1_MCLK: U?.E10 (SAI1_MCLK)
- new net SAI1_TXC: U?.C11 (SAI1_TXC)
- new net SAI1_TXD: U?.E11 (SAI1_TXD)
- new net SAI1_TXFS: U?.D11 (SAI1_TXFS)
- new net SD1_CD: U?.C6 (~SD1_CD)
- new net SD1_CLK: U?.B5 (SD1_CLK)
- new net SD1_CMD: U?.C5 (SD1_CMD)
- new net SD1_DATA0: U?.A5 (SD1_DATA0)
- new net SD1_DATA1: U?.D6 (SD1_DATA1)
- new net SD1_DATA2: U?.A4 (SD1_DATA2)
- new net SD1_DATA3: U?.D5 (SD1_DATA3)
- new net SD1_VSELECT: U?.R1 (GPIO1_IO8)
- new net SD2_CLK: U?.E3 (SD2_CLK)
- new net SD2_CMD: U?.F6 (SD2_CMD)
- new net SD2_DATA0: U?.E4 (SD2_DATA0)
- new net SD2_DATA1: U?.E5 (SD2_DATA1)
- new net SD2_DATA2: U?.F5 (SD2_DATA2)
- new net SD2_DATA3: U?.E6 (SD2_DATA3)
- new net UART1_RXD: U?.L3 (UART1_RXD)
- new net UART1_TXD: U?.L4 (UART1_TXD)
- new net UART3_CTS: U?.M6 (UART3_CTS)
- new net UART3_RTS: U?.M5 (UART3_RTS)
- new net UART3_RXD: U?.M1 (UART3_RXD)
- new net UART3_TXD: U?.M2 (UART3_TXD)
- new net USB_SUSPEND: U?.Y8 (SNVS_TAMPER1)
- new net WL_PMU_EN: U?.T5 (GPIO_IO14)
- new net WL_WAKE_AP: U?.T6 (GPIO_IO15)
- new net ~LCD_PWR_EN: U?.R2 (GPIO1_IO9)
- new net ~SD_PWR_EN: U?.R5 (GPIO1_IO10)
- no-connect marks 0 -> 78
Other:
- note added: "BOOTMODE[1:0]: 00 - Boot from fuses 01 - Serial Downloader 10 - Internal Boot 11 - Reserved"
- note added: "Configure as 32kHz clock output"
- note added: "There are already lot of decoupling caps just next to it."
- note added: "To Audio DAC"
- note added: "To SD card"
- note added: "To WiFi & BT"
- note added: "To WiFi&BT"

Commit message: - pcb: working on r0p1 sch
Parts:
- removed R?: 10K, Resistor_SMD:R_0603_1608Metric, symbol Device:R
- added R? (x2): 10K, Resistor_SMD:R_0603_1608Metric, symbol Device:R
- added R?: 4.7K/1%, Resistor_SMD:R_0603_1608Metric, symbol Device:R
Connections:
- net ADC1_IN0 is gone; now on net GND: U?.AD1 (ADC1_IN0)
- net ADC1_IN1 is gone; now on net GND: U?.AD3 (ADC1_IN1)
- net +1V8: now also C?.1, U?.L9 (NVCC_SPI); no longer C?.1, C?.1, C?.1, U?.F12 (NVCC_SAI), U?.L17 (NVCC_EPDC2), U?.M18 (NVCC_EPDC1)
- net +3V3: now also C?.1, C?.1, C?.1, U?.F12 (NVCC_SAI), U?.L17 (NVCC_EPDC2), U?.M18 (NVCC_EPDC1), R?.1, R?.1; no longer C?.1, U?.L9 (NVCC_SPI)
- net EPDC_BDR0: now also U?.K24 (EPDC_BDR0)
- net EPDC_D0: now also U?.P20 (EPDC_D0)
- net EPDC_D1: now also U?.P21 (EPDC_D1)
- net EPDC_D10: now also U?.L24 (EPDC_D10)
- net EPDC_D11: now also U?.L23 (EPDC_D11)
- net EPDC_D12: now also U?.L22 (EPDC_D12)
- net EPDC_D13: now also U?.L21 (EPDC_D13)
- net EPDC_D14: now also U?.L20 (EPDC_D14)
- net EPDC_D15: now also U?.K25 (EPDC_D15)
- net EPDC_D2: now also U?.N20 (EPDC_D2)
- net EPDC_D3: now also U?.N21 (EPDC_D3)
- net EPDC_D4: now also U?.N22 (EPDC_D4)
- net EPDC_D5: now also U?.M20 (EPDC_D5)
- net EPDC_D6: now also U?.M21 (EPDC_D6)
- net EPDC_D7: now also U?.M22 (EPDC_D7)
- net EPDC_D8: now also U?.M23 (EPDC_D8)
- net EPDC_D9: now also U?.L25 (EPDC_D9)
- net EPDC_GDCLK: now also U?.J25 (EPDC_GDCLK)
- net EPDC_GDOE: now also U?.J24 (EPDC_GDOE)
- net EPDC_GDSP: now also U?.H25 (EPDC_GDSP)
- net EPDC_PWRSTAT: now also U?.K20 (EPDC_PWRSTAT)
- net EPDC_SDCE0: now also U?.G25 (EPDC_SDCE0)
- net EPDC_SDCLK: now also U?.J21 (EPDC_SDCLK)
- net EPDC_SDLE: now also U?.J20 (EPDC_SDLE)
- net EPDC_SDOE: now also U?.H21 (EPDC_SDOE)
- net GND: now also U?.AE2 (ADC1_IN2), U?.AE3 (ADC1_IN3), R?.1; no longer U?.AA13 (PCIE_REXT)
- net USB_OTG_ID: now reaches U?.B7 (USB_OTG1_ID)
- net I2C2_SCL: now reaches U?.K2 (I2C2_SCL)
- net I2C2_SCL: now also R?.2
- net I2C2_SDA: now reaches U?.K3 (I2C2_SDA)
- net I2C2_SDA: now also R?.2
- net USB_HOST_DN: now reaches U?.A10 (USB_OTG2_DN)
- net USB_OTG_DN: now reaches U?.A8 (USB_OTG1_DN)
- net USB_HOST_DP: now reaches U?.B10 (USB_OTG2_DP)
- net USB_OTG_DP: now reaches U?.B8 (USB_OTG1_DP)
- net USB_HOST_VBUS: now reaches U?.C10 (USB2_VBUS)
- net USB_OTG_VBUS: now reaches U?.C8 (USB_OTG1_VBUS)
- net SAI1_RXD: now reaches U?.E12 (SAI1_RXD)
- net BAT_LOW: no longer names the net of U?.Y3 (SNVS_TAMPER9)
- net EXT_PWR_GOOD: no longer names the net of U?.AB6 (SNVS_TAMPER2)
- net POR renamed MPU_RST
- net SD1_CD: no longer names the net of U?.C6 (~SD1_CD)
- net USB_SUSPEND: no longer names the net of U?.Y8 (SNVS_TAMPER1)
- net ~LCD_PWR_EN: no longer names the net of U?.R2 (GPIO1_IO9)
- net ~SD_PWR_EN: no longer names the net of U?.R5 (GPIO1_IO10)
- new net: R?.2, U?.AA13 (PCIE_REXT)
- no-connect marks 78 -> 85
Other:
- note added: "BORDER"
- note added: "CKV"
- note added: "MODE"
- note added: "SPV"
- note added: "XCL"
- note added: "XLE"
- note added: "XOE"
- note added: "XSTL"

Commit message: - pcb: r0p1 sch draft
Parts:
- gave numbers to parts that had none: 48

Commit message: - pcb: start r0p1 layout
Parts:
- R101, R102, R103, R104, R105, R106, R107, R108, R109, R110, R111, R112, R113, R114, R115: footprint Resistor_SMD:R_0603_1608Metric -> Resistor_SMD:R_0402_1005Metric
Connections:
- net LCD_PWM: now reaches U101.N2 (GPIO1_IO1)
Other:
- company: Copyright EI-2030 2021. -> Copyright EI-2030 2021. / Engineer: Wenting Zhang
- title: Archer -> Archer Mainboard
Changed lines of the file:
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@@
   (paper "A3")
   (title_block
-    (title "Archer")
-    (date "2021-04-26")
+    (title "Archer Mainboard")
+    (date "2021-05-05")
     (rev "R0.1 draft")
-    (company "Copyright EI-2030 2021.")
+    (company "Copyright EI-2030 2021. / Engineer: Wenting Zhang")
     (comment 2 "MERCHANTABILITY, SATISFACTORY QUALITY AND FITNESS FOR A PARTICULAR PURPOSE.")
-    (comment 3 "source is distributed WITHOUT ANY EXPRESS OR IMPLIED WARRANTY, INCLUDING OF")
-    (comment 4 "This source describes Open Hardware and is licensed under the CERN-OHL-S v2. This ")
+    (comment 3 "This source is distributed WITHOUT ANY EXPRESS OR IMPLIED WARRANTY, INCLUDING OF")
+    (comment 4 "This source describes Open Hardware and is licensed under the CERN-OHL-S v2.")
   )
   (junction (at 26.67 31.75) (diameter 0.9144) (color 0 0 0 0))
@@
     (stroke (width 0) (type solid) (color 0 0 0 0))
   )
+  (wire (pts (xy 72.39 227.33) (xy 77.47 227.33))
+    (stroke (width 0) (type solid) (color 0 0 0 0))
+  )
   (wire (pts (xy 72.39 247.65) (xy 77.47 247.65))
     (stroke (width 0) (type solid) (color 0 0 0 0))
@@
   (label "MPU_JTAG_TRST" (at 193.04 200.66 0)
     (effects (font (size 1.27 1.27)) (justify left bottom))
+  )
+  (global_label "LCD_PWM" (shape output) (at 77.47 227.33 0) (fields_autoplaced)
+    (effects (font (size 1.27 1.27)) (justify left))
+    (property "Intersheet References" "${INTERSHEET_REFS}" (id 0) (at 88.5917 227.2506 0)
+      (effects (font (size 1.27 1.27)) (justify left) hide)
+    )
   )
   (global_label "SD1_VSELECT" (shape output) (at 77.47 247.65 0) (fields_autoplaced)
@@
     (property "Reference" "R101" (id 0) (at 121.92 185.42 90))
     (property "Value" "10K" (id 1) (at 121.92 193.04 90))
-    (property "Footprint" "Resistor_SMD:R_0603_1608Metric" (id 2) (at 121.158 189.23 90)
+    (property "Footprint" "Resistor_SMD:R_0402_1005Metric" (id 2) (at 121.158 189.23 90)
       (effects (font (size 1.27 1.27)) hide)
     )
@@
     (property "Reference" "R102" (id 0) (at 121.92 200.66 90))
     (property "Value" "DNP/10K" (id 1) (at 121.92 208.28 90))
-    (property "Footprint" "Resistor_SMD:R_0603_1608Metric" (id 2) (at 121.158 204.47 90)
+    (property "Footprint" "Resistor_SMD:R_0402_1005Metric" (id 2) (at 121.158 204.47 90)
       (effects (font (size 1.27 1.27)) hide)
     )
@@
     (property "Reference" "R103" (id 0) (at 127 185.42 90))
     (property "Value" "DNP/10K" (id 1) (at 127 193.04 90))
-    (property "Footprint" "Resistor_SMD:R_0603_1608Metric" (id 2) (at 126.238 189.23 90)
+    (property "Footprint" "Resistor_SMD:R_0402_1005Metric" (id 2) (at 126.238 189.23 90)
       (effects (font (size 1.27 1.27)) hide)
     )
@@
     (property "Reference" "R104" (id 0) (at 127 200.66 90))
     (property "Value" "10K" (id 1) (at 127 208.28 90))
-    (property "Footprint" "Resistor_SMD:R_0603_1608Metric" (id 2) (at 126.238 204.47 90)
+    (property "Footprint" "Resistor_SMD:R_0402_1005Metric" (id 2) (at 126.238 204.47 90)
       (effects (font (size 1.27 1.27)) hide)
     )
@@
       (effects (font (size 1.27 1.27)) (justify left))
     )
-    (property "Footprint" "Resistor_SMD:R_0603_1608Metric" (id 2) (at 186.182 24.13 90)
+    (property "Footprint" "Resistor_SMD:R_0402_1005Metric" (id 2) (at 186.182 24.13 90)
       (effects (font (size 1.27 1.27)) hide)
     )
@@
       (effects (font (size 1.27 1.27)) (justify right))
     )
-    (property "Footprint" "Resistor_SMD:R_0603_1608Metric" (id 2) (at 191.008 168.91 90)
+    (property "Footprint" "Resistor_SMD:R_0402_1005Metric" (id 2) (at 191.008 168.91 90)
       (effects (font (size 1.27 1.27)) hide)
     )
@@
       (effects (font (size 1.27 1.27)) (justify left))
     )
-    (property "Footprint" "Resistor_SMD:R_0603_1608Metric" (id 2) (at 193.802 24.13 90)
+    (property "Footprint" "Resistor_SMD:R_0402_1005Metric" (id 2) (at 193.802 24.13 90)
       (effects (font (size 1.27 1.27)) hide)
     )
@@
       (effects (font (size 1.27 1.27)) (justify left))
     )
-    (property "Footprint" "Resistor_SMD:R_0603_1608Metric" (id 2) (at 201.422 24.13 90)
+    (property "Footprint" "Resistor_SMD:R_0402_1005Metric" (id 2) (at 201.422 24.13 90)
       (effects (font (size 1.27 1.27)) hide)
     )
@@
     (property "Reference" "R109" (id 0) (at 209.55 238.5822 90))
     (property "Value" "1M" (id 1) (at 209.55 240.8936 90))
-    (property "Footprint" "Resistor_SMD:R_0603_1608Metric" (id 2) (at 209.55 242.062 90)
+    (property "Footprint" "Resistor_SMD:R_0402_1005Metric" (id 2) (at 209.55 242.062 90)
       (effects (font (size 1.27 1.27)) hide)
     )
@@
       (effects (font (size 1.27 1.27)) (justify left))
     )
-    (property "Footprint" "Resistor_SMD:R_0603_1608Metric" (id 2) (at 209.042 24.13 90)
+    (property "Footprint" "Resistor_SMD:R_0402_1005Metric" (id 2) (at 209.042 24.13 90)
       (effects (font (size 1.27 1.27)) hide)
     )
@@
     (property "Reference" "R111" (id 0) (at 232.41 230.9622 90))
     (property "Value" "DNP/4.75M" (id 1) (at 232.41 233.2736 90))
-    (property "Footprint" "Resistor_SMD:R_0603_1608Metric" (id 2) (at 232.41 234.442 90)
+    (property "Footprint" "Resistor_SMD:R_0402_1005Metric" (id 2) (at 232.41 234.442 90)
       (effects (font (size 1.27 1.27)) hide)
     )
@@
     (property "Reference" "R112" (id 0) (at 292.1 190.5 90))
     (property "Value" "200/1%" (id 1) (at 306.07 190.5 90))
-    (property "Footprint" "Resistor_SMD:R_0603_1608Metric" (id 2) (at 298.45 189.992 90)
+    (property "Footprint" "Resistor_SMD:R_0402_1005Metric" (id 2) (at 298.45 189.992 90)
       (effects (font (size 1.27 1.27)) hide)
     )
@@
     (property "Reference" "R113" (id 0) (at 292.1 203.2 90))
     (property "Value" "10K" (id 1) (at 306.07 203.2 90))
-    (property "Footprint" "Resistor_SMD:R_0603_1608Metric" (id 2) (at 298.45 202.692 90)
+    (property "Footprint" "Resistor_SMD:R_0402_1005Metric" (id 2) (at 298.45 202.692 90)
       (effects (font (size 1.27 1.27)) hide)
     )
@@
     (property "Reference" "R114" (id 0) (at 292.1 210.82 90))
     (property "Value" "200/1%" (id 1) (at 306.07 210.82 90))
-    (property "Footprint" "Resistor_SMD:R_0603_1608Metric" (id 2) (at 298.45 210.312 90)
+    (property "Footprint" "Resistor_SMD:R_0402_1005Metric" (id 2) (at 298.45 210.312 90)
       (effects (font (size 1.27 1.27)) hide)
     )
@@
       (effects (font (size 1.27 1.27)) (justify right))
     )
-    (property "Footprint" "Resistor_SMD:R_0603_1608Metric" (id 2) (at 386.588 133.35 90)
-      (effects (font (size 1.27 1.27)) hide)
-    )
+    (property "Footprint" "Resistor_SMD:R_0402_1005Metric" (id 2) (at 386.588 133.35 90)
+      (effects (font (size 1.27 1.27)) hide)
+    )

Commit message: - pcb: components placed
Connections:
- net PCIE_CLK_P: now reaches U101.AB10 (PCIE_REFCLKOUT_P)
- net PCIE_TX_P: now reaches U101.AB11 (PCIE_TX_P)
- net PCIE_CLK_N: now reaches U101.AC10 (PCIE_REFCLKOUT_N)
- net PCIE_TX_N: now reaches U101.AC11 (PCIE_TX_N)
- net PCIE_REFCLKIN_P: now reaches U101.AD10 (PCIE_REFCLKIN_P)
- net PCIE_RX_P: now reaches U101.AD11 (PCIE_RX_P)
- net PCIE_REFCLKIN_N: now reaches U101.AE10 (PCIE_REFCLKIN_N)
- net PCIE_RX_N: now reaches U101.AE11 (PCIE_RX_N)
- net +RTC renamed +3V3_SB
Changed lines of the file:
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@@
   (title_block
     (title "Archer Mainboard")
-    (date "2021-05-05")
+    (date "2021-05-06")
     (rev "R0.1 draft")
     (company "Copyright EI-2030 2021. / Engineer: Wenting Zhang")
@@
   (no_connect (at 382.27 77.47))
   (no_connect (at 382.27 80.01))
-  (no_connect (at 382.27 96.52))
-  (no_connect (at 382.27 99.06))
-  (no_connect (at 382.27 104.14))
-  (no_connect (at 382.27 106.68))
-  (no_connect (at 382.27 111.76))
-  (no_connect (at 382.27 114.3))
-  (no_connect (at 382.27 119.38))
-  (no_connect (at 382.27 121.92))
   (no_connect (at 382.27 143.51))
   (no_connect (at 382.27 146.05))
@@
   (no_connect (at 382.27 181.61))
   (no_connect (at 382.27 184.15))
+  (no_connect (at 400.05 96.52))
+  (no_connect (at 400.05 99.06))
+  (no_connect (at 400.05 104.14))
+  (no_connect (at 400.05 106.68))
+  (no_connect (at 400.05 111.76))
+  (no_connect (at 400.05 114.3))
+  (no_connect (at 400.05 119.38))
+  (no_connect (at 400.05 121.92))
   (wire (pts (xy 26.67 31.75) (xy 26.67 36.83))
     (stroke (width 0) (type solid) (color 0 0 0 0))
@@
   )
   (wire (pts (xy 381 247.65) (xy 378.46 247.65))
+    (stroke (width 0) (type solid) (color 0 0 0 0))
+  )
+  (wire (pts (xy 382.27 96.52) (xy 400.05 96.52))
+    (stroke (width 0) (type solid) (color 0 0 0 0))
+  )
+  (wire (pts (xy 382.27 99.06) (xy 400.05 99.06))
+    (stroke (width 0) (type solid) (color 0 0 0 0))
+  )
+  (wire (pts (xy 382.27 104.14) (xy 400.05 104.14))
+    (stroke (width 0) (type solid) (color 0 0 0 0))
+  )
+  (wire (pts (xy 382.27 106.68) (xy 400.05 106.68))
+    (stroke (width 0) (type solid) (color 0 0 0 0))
+  )
+  (wire (pts (xy 382.27 111.76) (xy 400.05 111.76))
+    (stroke (width 0) (type solid) (color 0 0 0 0))
+  )
+  (wire (pts (xy 382.27 114.3) (xy 400.05 114.3))
+    (stroke (width 0) (type solid) (color 0 0 0 0))
+  )
+  (wire (pts (xy 382.27 119.38) (xy 400.05 119.38))
+    (stroke (width 0) (type solid) (color 0 0 0 0))
+  )
+  (wire (pts (xy 382.27 121.92) (xy 400.05 121.92))
     (stroke (width 0) (type solid) (color 0 0 0 0))
   )
@@
   )
   (label "MPU_JTAG_TRST" (at 193.04 200.66 0)
+    (effects (font (size 1.27 1.27)) (justify left bottom))
+  )
+  (label "PCIE_REFCLKIN_P" (at 384.81 96.52 0)
+    (effects (font (size 1.27 1.27)) (justify left bottom))
+  )
+  (label "PCIE_REFCLKIN_N" (at 384.81 99.06 0)
+    (effects (font (size 1.27 1.27)) (justify left bottom))
+  )
+  (label "PCIE_CLK_P" (at 384.81 104.14 0)
+    (effects (font (size 1.27 1.27)) (justify left bottom))
+  )
+  (label "PCIE_CLK_N" (at 384.81 106.68 0)
+    (effects (font (size 1.27 1.27)) (justify left bottom))
+  )
+  (label "PCIE_RX_P" (at 384.81 111.76 0)
+    (effects (font (size 1.27 1.27)) (justify left bottom))
+  )
+  (label "PCIE_RX_N" (at 384.81 114.3 0)
+    (effects (font (size 1.27 1.27)) (justify left bottom))
+  )
+  (label "PCIE_TX_P" (at 384.81 119.38 0)
+    (effects (font (size 1.27 1.27)) (justify left bottom))
+  )
+  (label "PCIE_TX_N" (at 384.81 121.92 0)
     (effects (font (size 1.27 1.27)) (justify left bottom))
   )
@@
     (pin "1")
   )
-  (symbol (lib_id "symbols:+RTC") (at 124.46 180.34 0) (unit 1)
+  (symbol (lib_id "symbols:+3V3_SB") (at 124.46 180.34 0) (unit 1)
     (in_bom yes) (on_board yes)
     (property "Reference" "#PWR0110" (id 0) (at 124.46 184.15 0)
       (effects (font (size 1.27 1.27)) hide)
     )
-    (property "Value" "+RTC" (id 1) (at 124.841 175.9458 0))
+    (property "Value" "+3V3_SB" (id 1) (at 120.0151 176.53 0)
+      (effects (font (size 1.27 1.27)) (justify left))
+    )
     (property "Footprint" "" (id 2) (at 124.46 180.34 0)
       (effects (font (size 1.27 1.27)) hide)
