File: pcb/mainboard/cpu.kicad_sch (KiCad schematic)
At the start: 48 parts, among them U101 MCIMX7S5EVM08SC, Y101 24MHz, Y102 32.768kHz

Commit message: - pcb: finishing layout r0p1
Connections:
- net USB_HOST_VBUS is gone; now on net +3V3: U101.C10 (USB2_VBUS)
- net USB_OTG_VBUS is gone; now on net +3V3: U101.C8 (USB_OTG1_VBUS)
- net BT_CFG_1: now also RN101.3 (R3.1); no longer RN101.4 (R4.1)
- net BT_CFG_12: now also RN101.4 (R4.1); no longer RN101.2 (R2.1)
- net BT_CFG_4: now also RN101.2 (R2.1); no longer RN101.3 (R3.1)
- net LCD_TP_INT: now reaches U101.P1 (GPIO1_IO5)
- net EPD_TP_INT: now reaches U101.P2 (GPIO1_IO6)
- net EPD_PWR_EN: now reaches U101.L1 (I2C4_SCL)
- net +VCCIO_WL renamed +VCCIO_SD
- net PB_STAT renamed ONOFF
Changed lines of the file:
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@@
+    (stroke (width 0) (type solid) (color 0 0 0 0))
+  )
+  (wire (pts (xy 72.39 237.49) (xy 77.47 237.49))
+    (stroke (width 0) (type solid) (color 0 0 0 0))
+  )
+  (wire (pts (xy 72.39 240.03) (xy 77.47 240.03))
     (stroke (width 0) (type solid) (color 0 0 0 0))
   )
@@
     (stroke (width 0) (type solid) (color 0 0 0 0))
   )
+  (wire (pts (xy 185.42 53.34) (xy 190.5 53.34))
+    (stroke (width 0) (type solid) (color 0 0 0 0))
+  )
   (wire (pts (xy 185.42 86.36) (xy 190.5 86.36))
     (stroke (width 0) (type solid) (color 0 0 0 0))
@@
     (stroke (width 0) (type solid) (color 0 0 0 0))
   )
-  (wire (pts (xy 347.98 209.55) (xy 363.22 209.55))
+  (wire (pts (xy 347.98 209.55) (xy 360.68 209.55))
     (stroke (width 0) (type solid) (color 0 0 0 0))
   )
@@
     (stroke (width 0) (type solid) (color 0 0 0 0))
   )
-  (wire (pts (xy 347.98 217.17) (xy 360.68 217.17))
+  (wire (pts (xy 347.98 217.17) (xy 358.14 217.17))
     (stroke (width 0) (type solid) (color 0 0 0 0))
   )
@@
     (stroke (width 0) (type solid) (color 0 0 0 0))
   )
-  (wire (pts (xy 347.98 229.87) (xy 358.14 229.87))
+  (wire (pts (xy 347.98 229.87) (xy 365.76 229.87))
     (stroke (width 0) (type solid) (color 0 0 0 0))
   )
@@
     (stroke (width 0) (type solid) (color 0 0 0 0))
   )
-  (wire (pts (xy 358.14 229.87) (xy 358.14 207.01))
+  (wire (pts (xy 358.14 217.17) (xy 358.14 207.01))
     (stroke (width 0) (type solid) (color 0 0 0 0))
   )
@@
     (stroke (width 0) (type solid) (color 0 0 0 0))
   )
-  (wire (pts (xy 360.68 217.17) (xy 360.68 207.01))
+  (wire (pts (xy 360.68 209.55) (xy 360.68 207.01))
     (stroke (width 0) (type solid) (color 0 0 0 0))
   )
@@
     (stroke (width 0) (type solid) (color 0 0 0 0))
   )
-  (wire (pts (xy 363.22 209.55) (xy 363.22 207.01))
-    (stroke (width 0) (type solid) (color 0 0 0 0))
-  )
   (wire (pts (xy 363.22 224.79) (xy 363.22 237.49))
     (stroke (width 0) (type solid) (color 0 0 0 0))
   )
   (wire (pts (xy 363.22 247.65) (xy 360.68 247.65))
+    (stroke (width 0) (type solid) (color 0 0 0 0))
+  )
+  (wire (pts (xy 365.76 207.01) (xy 363.22 207.01))
+    (stroke (width 0) (type solid) (color 0 0 0 0))
+  )
+  (wire (pts (xy 365.76 229.87) (xy 365.76 207.01))
     (stroke (width 0) (type solid) (color 0 0 0 0))
   )
@@
     )
   )
+  (global_label "LCD_TP_INT" (shape input) (at 77.47 237.49 0) (fields_autoplaced)
+    (effects (font (size 1.27 1.27)) (justify left))
+    (property "Intersheet References" "${INTERSHEET_REFS}" (id 0) (at 90.5269 237.4106 0)
+      (effects (font (size 1.27 1.27)) (justify left) hide)
+    )
+  )
+  (global_label "EPD_TP_INT" (shape input) (at 77.47 240.03 0) (fields_autoplaced)
+    (effects (font (size 1.27 1.27)) (justify left))
+    (property "Intersheet References" "${INTERSHEET_REFS}" (id 0) (at 90.6479 239.9506 0)
+      (effects (font (size 1.27 1.27)) (justify left) hide)
+    )
+  )
   (global_label "SD1_VSELECT" (shape output) (at 77.47 247.65 0) (fields_autoplaced)
     (effects (font (size 1.27 1.27)) (justify left))
@@
     )
   )
-  (global_label "PB_STAT" (shape input) (at 142.24 187.96 180) (fields_autoplaced)
+  (global_label "ONOFF" (shape input) (at 142.24 187.96 180) (fields_autoplaced)
     (effects (font (size 1.27 1.27)) (justify right))
-    (property "Intersheet References" "${INTERSHEET_REFS}" (id 0) (at 99.06 151.13 0)
-      (effects (font (size 1.27 1.27)) hide)
+    (property "Intersheet References" "${INTERSHEET_REFS}" (id 0) (at 133.6583 187.8806 0)
+      (effects (font (size 1.27 1.27)) (justify right) hide)
     )
   )
@@
     )
   )
+  (global_label "EPD_PWR_EN" (shape output) (at 190.5 53.34 0)
+    (effects (font (size 1.27 1.27)) (justify left))
+    (property "Intersheet References" "${INTERSHEET_REFS}" (id 0) (at 294.64 167.64 0)
+      (effects (font (size 1.27 1.27)) hide)
+    )
+  )
   (global_label "UART1_RXD" (shape input) (at 190.5 86.36 0) (fields_autoplaced)
     (effects (font (size 1.27 1.27)) (justify left))
@@
     )
   )
-  (global_label "USB_OTG_VBUS" (shape input) (at 292.1 184.15 0) (fields_autoplaced)
-    (effects (font (size 1.27 1.27)) (justify left))
-    (property "Intersheet References" "${INTERSHEET_REFS}" (id 0) (at 308.725 184.0706 0)
-      (effects (font (size 1.27 1.27)) (justify left) hide)
-    )
-  )
   (global_label "USB_HOST_DP" (shape bidirectional) (at 292.1 196.85 0) (fields_autoplaced)
     (effects (font (size 1.27 1.27)) (justify left))
@@
     (effects (font (size 1.27 1.27)) (justify left))
     (property "Intersheet References" "${INTERSHEET_REFS}" (id 0) (at 307.6969 199.3106 0)
-      (effects (font (size 1.27 1.27)) (justify left) hide)
-    )
-  )
-  (global_label "USB_HOST_VBUS" (shape input) (at 292.1 207.01 0) (fields_autoplaced)
-    (effects (font (size 1.27 1.27)) (justify left))
-    (property "Intersheet References" "${INTERSHEET_REFS}" (id 0) (at 309.995 206.9306 0)
       (effects (font (size 1.27 1.27)) (justify left) hide)
     )
@@
       (effects (font (size 1.27 1.27)) hide)
     )
+    (pin "1")
+  )
+  (symbol (lib_id "power:+3V3") (at 292.1 184.15 270) (unit 1)
+    (in_bom yes) (on_board yes)
+    (property "Reference" "#PWR0167" (id 0) (at 288.29 184.15 0)
+      (effects (font (size 1.27 1.27)) hide)
+    )
+    (property "Value" "+3V3" (id 1) (at 297.7642 184.531 90))
+    (property "Footprint" "" (id 2) (at 292.1 184.15 0)
+      (effects (font (size 1.27 1.27)) hide)
+    )
+    (property "Datasheet" "" (id 3) (at 292.1 184.15 0)
+      (effects (font (size 1.27 1.27)) hide)
+    )
+    (pin "1")
+  )
+  (symbol (lib_id "power:+3V3") (at 292.1 207.01 270) (unit 1)
+    (in_bom yes) (on_board yes)
+    (property "Reference" "#PWR0168" (id 0) (at 288.29 207.01 0)
+      (effects (font (size 1.27 1.27)) hide)
+    )
+    (property "Value" "+3V3" (id 1) (at 297.7642 207.391 90))
+    (property "Footprint" "" (id 2) (at 292.1 207.01 0)
+      (effects (font (size 1.27 1.27)) hide)
+    )
+    (property "Datasheet" "" (id 3) (at 292.1 207.01 0)
+      (effects (font (size 1.27 1.27)) hide)
+    )
