File: pcb/mainboard/ddr.kicad_sch (KiCad schematic)
At the start: 0 parts

Commit message: - pcb: switch to imx7 for the prototype
Parts:
- added C? (x19): 220nF, Capacitor_SMD:C_0402_1005Metric, symbol Device:C
- added C? (x5): 22uF, Capacitor_SMD:C_0603_1608Metric, symbol Device:C
- added C?: 4.7uF, Capacitor_SMD:C_0603_1608Metric, symbol Device:C
- added C? (x3): 100nF, Capacitor_SMD:C_0402_1005Metric, symbol Device:C
- added R?: 240R 1%, Resistor_SMD:R_0402_1005Metric, symbol Device:R
- added R? (x2): 1.5K/0.5%, Resistor_SMD:R_0402_1005Metric, symbol Device:R
- added U? (x2): MT41K256M16HA, Package_BGA:BGA-96_9.0x13.0mm_Layout2x3x16_P0.8mm, symbol symbols:MT41K256M16HA
- added U?: MCIMX7S5EVM08SC, footprints:BGA-541_25x25_19.0x19.0mm, symbol symbols:MCIMX7S5EVM08SC
Connections:
- new net: R?.2, U?.AB13 (DRAM_ZQPAD)
- new net +1V2: C?.1, C?.1, C?.1, C?.1, C?.1, C?.1, C?.1, C?.1, C?.1, C?.1, C?.1, C?.1, C?.1, C?.1, C?.1, C?.1, C?.1, C?.1, C?.1, C?.1, C?.1, C?.1, C?.1, R?.1, U?.AA16 (NVCC_DRAM), U?.AA17 (NVCC_DRAM), U?.AA18 (NVCC_DRAM), U?.AA19 (NVCC_DRAM), U?.AA20 (NVCC_DRAM), U?.AA21 (NVCC_DRAM), U?.T21 (NVCC_DRAM), U?.U21 (NVCC_DRAM), U?.V21 (NVCC_DRAM), U?.W21 (NVCC_DRAM), U?.Y20 (NVCC_DRAM_CKE), U?.Y21 (NVCC_DRAM)
- new net +DRAM_1V8: C?.1, C?.1, C?.1
- new net +DRAM_VREF: C?.1, C?.1, C?.2, R?.1, R?.2, U?.AC13 (DRAM_VREF)
- new net DRAM_ADDR0: U?.AB19 (DRAM_ADDR0), U?.N3 (A0), U?.N3 (A0)
- new net DRAM_ADDR1: U?.AB16 (DRAM_ADDR1), U?.P7 (A1), U?.P7 (A1)
- new net DRAM_ADDR10: U?.L7 (A10), U?.L7 (A10), U?.T23 (DRAM_ADDR10)
- new net DRAM_ADDR11: U?.R7 (A11), U?.R7 (A11), U?.U22 (DRAM_ADDR11)
- new net DRAM_ADDR12: U?.N7 (A12/~BC), U?.N7 (A12/~BC), U?.T22 (DRAM_ADDR12)
- new net DRAM_ADDR13: U?.P23 (DRAM_ADDR13), U?.T3 (A13), U?.T3 (A13)
- new net DRAM_ADDR14: U?.AB18 (DRAM_ADDR14), U?.T7 (A14/NC), U?.T7 (A14/NC)
- new net DRAM_ADDR2: U?.AC18 (DRAM_ADDR2), U?.P3 (A2), U?.P3 (A2)
- new net DRAM_ADDR3: U?.AC20 (DRAM_ADDR3), U?.N2 (A3), U?.N2 (A3)
- new net DRAM_ADDR4: U?.AB21 (DRAM_ADDR4), U?.P8 (A4), U?.P8 (A4)
- new net DRAM_ADDR5: U?.P2 (A5), U?.P2 (A5), U?.Y23 (DRAM_ADDR5)
- new net DRAM_ADDR6: U?.R8 (A6), U?.R8 (A6), U?.V22 (DRAM_ADDR6)
- new net DRAM_ADDR7: U?.R2 (A7), U?.R2 (A7), U?.Y22 (DRAM_ADDR7)
- new net DRAM_ADDR8: U?.T8 (A8), U?.T8 (A8), U?.W22 (DRAM_ADDR8)
- new net DRAM_ADDR9: U?.R3 (A9), U?.R3 (A9), U?.V23 (DRAM_ADDR9)
- new net DRAM_BA0: U?.M2 (BA0), U?.M2 (BA0), U?.R22 (DRAM_SDBA0)
- new net DRAM_BA1: U?.N8 (BA1), U?.N8 (BA1), U?.P22 (DRAM_SDBA1)
- new net DRAM_BA2: U?.M3 (BA2), U?.M3 (BA2), U?.N23 (DRAM_SDBA2)
- new net DRAM_CASB: U?.AC14 (~DRAM_CAS), U?.K3 (~CAS), U?.K3 (~CAS)
- new net DRAM_CKE: U?.AB17 (DRAM_SDCKE0), U?.K9 (CKE), U?.K9 (CKE)
- new net DRAM_CKN: U?.AD25 (DRAM_SDCLK0_N), U?.K7 (~CK), U?.K7 (~CK)
- new net DRAM_CKP: U?.AD24 (DRAM_SDCLK0_P), U?.J7 (CK), U?.J7 (CK)
- new net DRAM_CSB: U?.AB23 (~DRAM_CS0), U?.L2 (~CS), U?.L2 (~CS)
- new net DRAM_DATA0: U?.A7 (DQ12), U?.AD22 (DRAM_DATA0)
- new net DRAM_DATA1: U?.A3 (DQ15), U?.AD23 (DRAM_DATA1)
- new net DRAM_DATA10: U?.AE17 (DRAM_DATA10), U?.F2 (DQ2)
- new net DRAM_DATA11: U?.AD16 (DRAM_DATA11), U?.H3 (DQ4)
- new net DRAM_DATA12: U?.AE16 (DRAM_DATA12), U?.H8 (DQ5)
- new net DRAM_DATA13: U?.AD14 (DRAM_DATA13), U?.F8 (DQ3)
- new net DRAM_DATA14: U?.AD13 (DRAM_DATA14), U?.F7 (DQ1)
- new net DRAM_DATA15: U?.AE13 (DRAM_DATA15), U?.H7 (DQ7)
- new net DRAM_DATA16: U?.AA25 (DRAM_DATA16), U?.G2 (DQ6)
- new net DRAM_DATA17: U?.E3 (DQ0), U?.W24 (DRAM_DATA17)
- new net DRAM_DATA18: U?.F2 (DQ2), U?.V25 (DRAM_DATA18)
- new net DRAM_DATA19: U?.H3 (DQ4), U?.W25 (DRAM_DATA19)
- new net DRAM_DATA2: U?.AE20 (DRAM_DATA2), U?.C2 (DQ11)
- new net DRAM_DATA20: U?.AC25 (DRAM_DATA20), U?.F8 (DQ3)
- new net DRAM_DATA21: U?.AB25 (DRAM_DATA21), U?.F7 (DQ1)
- new net DRAM_DATA22: U?.AB24 (DRAM_DATA22), U?.H8 (DQ5)
- new net DRAM_DATA23: U?.AC24 (DRAM_DATA23), U?.H7 (DQ7)
- new net DRAM_DATA24: U?.A2 (DQ13), U?.R25 (DRAM_DATA24)
- new net DRAM_DATA25: U?.A7 (DQ12), U?.N24 (DRAM_DATA25)
- new net DRAM_DATA26: U?.C2 (DQ11), U?.P25 (DRAM_DATA26)
- new net DRAM_DATA27: U?.B8 (DQ14), U?.N25 (DRAM_DATA27)
- new net DRAM_DATA28: U?.D7 (DQ8), U?.U25 (DRAM_DATA28)
- new net DRAM_DATA29: U?.C8 (DQ10), U?.R24 (DRAM_DATA29)
- new net DRAM_DATA3: U?.A2 (DQ13), U?.AE23 (DRAM_DATA3)
- new net DRAM_DATA30: U?.A3 (DQ15), U?.U24 (DRAM_DATA30)
- new net DRAM_DATA31: U?.C3 (DQ9), U?.V24 (DRAM_DATA31)
- new net DRAM_DATA4: U?.AE22 (DRAM_DATA4), U?.D7 (DQ8)
- new net DRAM_DATA5: U?.AD19 (DRAM_DATA5), U?.B8 (DQ14)
- new net DRAM_DATA6: U?.AD18 (DRAM_DATA6), U?.C3 (DQ9)
- new net DRAM_DATA7: U?.AE19 (DRAM_DATA7), U?.C8 (DQ10)
- new net DRAM_DATA8: U?.AE14 (DRAM_DATA8), U?.G2 (DQ6)
- new net DRAM_DATA9: U?.AE18 (DRAM_DATA9), U?.E3 (DQ0)
- new net DRAM_DQM0: U?.AD20 (DRAM_DQM0), U?.D3 (UDM)
- new net DRAM_DQM1: U?.AD17 (DRAM_DQM1), U?.E7 (LDM)
- new net DRAM_DQM2: U?.AA24 (DRAM_DQM2), U?.E7 (LDM)
- new net DRAM_DQM3: U?.D3 (UDM), U?.P24 (DRAM_DQM3)
- new net DRAM_ODT: U?.AC16 (DRAM_ODT0), U?.K1 (ODT), U?.K1 (ODT)
- new net DRAM_RASB: U?.AB15 (~DRAM_RAS), U?.J3 (~RAS), U?.J3 (~RAS)
- new net DRAM_RST: U?.AC22 (DRAM_RESET), U?.T2 (~RESET), U?.T2 (~RESET)
- new net DRAM_SDQSN_0: U?.AD21 (DRAM_SDQS0_N), U?.B7 (~UDQS)
- new net DRAM_SDQSN_1: U?.AE15 (DRAM_SDQS1_N), U?.G3 (~LDQS)
- new net DRAM_SDQSN_2: U?.G3 (~LDQS), U?.Y25 (DRAM_SDQS2_N)
- new net DRAM_SDQSN_3: U?.B7 (~UDQS), U?.T25 (DRAM_SDQS3_N)
- new net DRAM_SDQSP_0: U?.AE21 (DRAM_SDQS0_P), U?.C7 (UDQS)
- new net DRAM_SDQSP_1: U?.AD15 (DRAM_SDQS1_P), U?.F3 (LDQS)
- new net DRAM_SDQSP_2: U?.F3 (LDQS), U?.Y24 (DRAM_SDQS2_P)
- new net DRAM_SDQSP_3: U?.C7 (UDQS), U?.T24 (DRAM_SDQS3_P)
- new net DRAM_WEB: U?.AB14 (~DRAM_SDWE), U?.L3 (~WE), U?.L3 (~WE)
- new net GND: C?.2, C?.2, C?.2, C?.2, C?.2, C?.2, C?.2, C?.2, C?.2, C?.2, C?.2, C?.2, C?.2, C?.2, C?.2, C?.2, C?.2, C?.2, C?.2, C?.2, C?.2, C?.2, C?.2, C?.2, C?.2, C?.2, C?.2, R?.1, R?.2
- new net VDD: U?.B2 (VDD), U?.B2 (VDD), U?.D9 (VDD), U?.D9 (VDD), U?.G7 (VDD), U?.G7 (VDD), U?.K2 (VDD), U?.K2 (VDD), U?.K8 (VDD), U?.K8 (VDD), U?.N1 (VDD), U?.N1 (VDD), U?.N9 (VDD), U?.N9 (VDD), U?.R1 (VDD), U?.R1 (VDD), U?.R9 (VDD), U?.R9 (VDD)
- new net VDDQ: U?.A1 (VDDQ), U?.A1 (VDDQ), U?.A8 (VDDQ), U?.A8 (VDDQ), U?.C1 (VDDQ), U?.C1 (VDDQ), U?.C9 (VDDQ), U?.C9 (VDDQ), U?.D2 (VDDQ), U?.D2 (VDDQ), U?.E9 (VDDQ), U?.E9 (VDDQ), U?.F1 (VDDQ), U?.F1 (VDDQ), U?.H2 (VDDQ), U?.H2 (VDDQ), U?.H9 (VDDQ), U?.H9 (VDDQ)
- new net VSS: U?.A9 (VSS), U?.A9 (VSS), U?.B3 (VSS), U?.B3 (VSS), U?.E1 (VSS), U?.E1 (VSS), U?.G8 (VSS), U?.G8 (VSS), U?.J2 (VSS), U?.J2 (VSS), U?.J8 (VSS), U?.J8 (VSS), U?.M1 (VSS), U?.M1 (VSS), U?.M9 (VSS), U?.M9 (VSS), U?.P1 (VSS), U?.P1 (VSS), U?.P9 (VSS), U?.P9 (VSS), U?.T1 (VSS), U?.T1 (VSS), U?.T9 (VSS), U?.T9 (VSS)
- new net VSSQ: U?.B1 (VSSQ), U?.B1 (VSSQ), U?.B9 (VSSQ), U?.B9 (VSSQ), U?.D1 (VSSQ), U?.D1 (VSSQ), U?.D8 (VSSQ), U?.D8 (VSSQ), U?.E2 (VSSQ), U?.E2 (VSSQ), U?.E8 (VSSQ), U?.E8 (VSSQ), U?.F9 (VSSQ), U?.F9 (VSSQ), U?.G1 (VSSQ), U?.G1 (VSSQ), U?.G9 (VSSQ), U?.G9 (VSSQ)
- no-connect marks 0 -> 2
Other:
- note added: "CAP for LPDDR_VDD1"
- note added: "CAP for LPDDR_VDD2"
- note added: "CAP for LPDDR_VDDCA"
- note added: "CAP for VDDQ"

Commit message: - pcb: working on r0p1 sch
Parts:
- removed C? (x4): 220nF, Capacitor_SMD:C_0402_1005Metric, symbol Device:C
- removed C? (x2): 22uF, Capacitor_SMD:C_0603_1608Metric, symbol Device:C
- added C? (x18): 220nF, Capacitor_SMD:C_0402_1005Metric, symbol Device:C
- added C? (x2): 22uF, Capacitor_SMD:C_0603_1608Metric, symbol Device:C
- added R? (x2): 240R 1%, Resistor_SMD:R_0402_1005Metric, symbol Device:R
- added R? (x2): 10K, Resistor_SMD:R_0402_1005Metric, symbol Device:R
Connections:
- net VDD is gone; now on net +1V35: U?.B2 (VDD), U?.B2 (VDD), U?.D9 (VDD), U?.D9 (VDD), U?.G7 (VDD), U?.G7 (VDD), U?.K2 (VDD), U?.K2 (VDD), U?.K8 (VDD), U?.K8 (VDD), U?.N1 (VDD), U?.N1 (VDD), U?.N9 (VDD), U?.N9 (VDD), U?.R1 (VDD), U?.R1 (VDD), U?.R9 (VDD), U?.R9 (VDD)
- net VDDQ is gone; now on net +1V35: U?.A1 (VDDQ), U?.A1 (VDDQ), U?.A8 (VDDQ), U?.A8 (VDDQ), U?.C1 (VDDQ), U?.C1 (VDDQ), U?.C9 (VDDQ), U?.C9 (VDDQ), U?.D2 (VDDQ), U?.D2 (VDDQ), U?.E9 (VDDQ), U?.E9 (VDDQ), U?.F1 (VDDQ), U?.F1 (VDDQ), U?.H2 (VDDQ), U?.H2 (VDDQ), U?.H9 (VDDQ), U?.H9 (VDDQ)
- net VSS is gone; now on net GND: U?.A9 (VSS), U?.A9 (VSS), U?.B3 (VSS), U?.B3 (VSS), U?.E1 (VSS), U?.E1 (VSS), U?.G8 (VSS), U?.G8 (VSS), U?.J2 (VSS), U?.J2 (VSS), U?.J8 (VSS), U?.J8 (VSS), U?.M1 (VSS), U?.M1 (VSS), U?.M9 (VSS), U?.M9 (VSS), U?.P1 (VSS), U?.P1 (VSS), U?.P9 (VSS), U?.P9 (VSS), U?.T1 (VSS), U?.T1 (VSS), U?.T9 (VSS), U?.T9 (VSS)
- net VSSQ is gone; now on net GND: U?.B1 (VSSQ), U?.B1 (VSSQ), U?.B9 (VSSQ), U?.B9 (VSSQ), U?.D1 (VSSQ), U?.D1 (VSSQ), U?.D8 (VSSQ), U?.D8 (VSSQ), U?.E2 (VSSQ), U?.E2 (VSSQ), U?.E8 (VSSQ), U?.E8 (VSSQ), U?.F9 (VSSQ), U?.F9 (VSSQ), U?.G1 (VSSQ), U?.G1 (VSSQ), U?.G9 (VSSQ), U?.G9 (VSSQ)
- net +1V2: no longer C?.1, C?.1, C?.1, C?.1, C?.1, C?.1, C?.1, C?.1, C?.1, C?.1, C?.1, C?.1, R?.1
- net +DRAM_VREF: now also U?.H1 (VrefDQ), U?.H1 (VrefDQ), U?.M8 (VrefCA), U?.M8 (VrefCA), C?.1, C?.1, C?.1, C?.1
- net DRAM_CKE: now also R?.2
- net DRAM_RST: now also R?.2
- net GND: now also C?.2, C?.2, C?.2, C?.2, C?.2, C?.2, C?.2, C?.2, C?.2, C?.2, C?.2, C?.2, C?.2, C?.2, C?.2, C?.2, C?.2, C?.2, C?.2, C?.2, R?.1, R?.1, R?.2, R?.2
- net at U?.L8 (ZQ): now also R?.1 (x2)
- net +DRAM_1V8 renamed +1V35
- net +1V35: now also C?.1, C?.1, C?.1, C?.1, C?.1, C?.1, C?.1, C?.1, C?.1, C?.1, C?.1, C?.1, R?.1, C?.1, C?.1, C?.1, C?.1, C?.1, C?.1, C?.1, C?.1, C?.1, C?.1, C?.1, C?.1, C?.1, C?.1, C?.1, C?.1
- no-connect marks 2 -> 6
Other:
- note added: "CAP for DRAM0"
- note added: "CAP for DRAM1"
- note removed: "CAP for LPDDR_VDD1"
- note removed: "CAP for LPDDR_VDD2"
- note removed: "CAP for LPDDR_VDDCA"
- note removed: "CAP for VDDQ"
- moved on the sheet: C?, R?

Commit message: - pcb: r0p1 sch draft
Parts:
- gave numbers to parts that had none: 52

Commit message: - pcb: start r0p1 layout
Parts:
- renumbered U201 to U101
Connections:
- net +1V2 is gone; now on net +1V35: C201.1, C202.1, C203.1, C204.1, C205.1, C207.1, U101.AA16 (NVCC_DRAM), U101.AA17 (NVCC_DRAM), U101.AA18 (NVCC_DRAM), U101.AA19 (NVCC_DRAM), U101.AA20 (NVCC_DRAM), U101.AA21 (NVCC_DRAM), U101.T21 (NVCC_DRAM), U101.U21 (NVCC_DRAM), U101.V21 (NVCC_DRAM), U101.W21 (NVCC_DRAM), U101.Y20 (NVCC_DRAM_CKE), U101.Y21 (NVCC_DRAM)
Other:
- company: Copyright EI-2030 2021. -> Copyright EI-2030 2021. / Engineer: Wenting Zhang
- title: Archer -> Archer Mainboard
Changed lines of the file:
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@@
   (paper "A3")
   (title_block
-    (title "Archer")
-    (date "2021-04-26")
+    (title "Archer Mainboard")
+    (date "2021-05-05")
     (rev "R0.1 draft")
-    (company "Copyright EI-2030 2021.")
+    (company "Copyright EI-2030 2021. / Engineer: Wenting Zhang")
     (comment 2 "MERCHANTABILITY, SATISFACTORY QUALITY AND FITNESS FOR A PARTICULAR PURPOSE.")
-    (comment 3 "source is distributed WITHOUT ANY EXPRESS OR IMPLIED WARRANTY, INCLUDING OF")
-    (comment 4 "This source describes Open Hardware and is licensed under the CERN-OHL-S v2. This ")
+    (comment 3 "This source is distributed WITHOUT ANY EXPRESS OR IMPLIED WARRANTY, INCLUDING OF")
+    (comment 4 "This source describes Open Hardware and is licensed under the CERN-OHL-S v2.")
   )
   (junction (at 30.48 195.58) (diameter 0.9144) (color 0 0 0 0))
@@
     (effects (font (size 1.27 1.27)) (justify left bottom))
   )
-  (symbol (lib_id "power:+1V2") (at 30.48 195.58 0) (unit 1)
-    (in_bom yes) (on_board yes)
-    (property "Reference" "#PWR0201" (id 0) (at 30.48 199.39 0)
+  (symbol (lib_id "power:+1V35") (at 30.48 195.58 0) (unit 1)
+    (in_bom yes) (on_board yes) (fields_autoplaced)
+    (property "Reference" "#PWR?" (id 0) (at 30.48 199.39 0)
       (effects (font (size 1.27 1.27)) hide)
     )
-    (property "Value" "+1V2" (id 1) (at 30.861 191.1858 0))
+    (property "Value" "+1V35" (id 1) (at 30.48 191.77 0))
     (property "Footprint" "" (id 2) (at 30.48 195.58 0)
       (effects (font (size 1.27 1.27)) hide)
@@
     (pin "1")
   )
-  (symbol (lib_id "power:+1V2") (at 162.56 205.74 0) (unit 1)
-    (in_bom yes) (on_board yes)
-    (property "Reference" "#PWR0208" (id 0) (at 162.56 209.55 0)
+  (symbol (lib_id "power:+1V35") (at 162.56 205.74 0) (unit 1)
+    (in_bom yes) (on_board yes) (fields_autoplaced)
+    (property "Reference" "#PWR?" (id 0) (at 162.56 209.55 0)
       (effects (font (size 1.27 1.27)) hide)
     )
-    (property "Value" "+1V2" (id 1) (at 162.941 201.3458 0))
+    (property "Value" "+1V35" (id 1) (at 162.56 201.93 0))
     (property "Footprint" "" (id 2) (at 162.56 205.74 0)
       (effects (font (size 1.27 1.27)) hide)
@@
   (symbol (lib_id "symbols:MCIMX7S5EVM08SC") (at 104.14 124.46 0) (unit 3)
     (in_bom yes) (on_board yes)
-    (property "Reference" "U201" (id 0) (at 88.9 67.31 0))
+    (property "Reference" "U101" (id 0) (at 88.9 67.31 0))
     (property "Value" "MCIMX7S5EVM08SC" (id 1) (at 113.03 67.31 0))
     (property "Footprint" "footprints:BGA-541_25x25_19.0x19.0mm" (id 2) (at 104.14 106.68 0)

Commit message: - pcb: finishing layout r0p1
Parts:
- U202, U203: footprint Package_BGA:BGA-96_9.0x13.0mm_Layout2x3x16_P0.8mm -> footprints:BGA-96_9.0x13.0mm_P0.8mm
Changed lines of the file:
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@@
       (effects (font (size 1.1938 1.1938)))
     )
-    (property "Footprint" "Package_BGA:BGA-96_9.0x13.0mm_Layout2x3x16_P0.8mm" (id 2) (at 248.92 39.37 0)
+    (property "Footprint" "footprints:BGA-96_9.0x13.0mm_P0.8mm" (id 2) (at 248.92 39.37 0)
       (effects (font (size 1.1938 1.1938)) hide)
     )
@@
       (effects (font (size 1.1938 1.1938)))
     )
-    (property "Footprint" "Package_BGA:BGA-96_9.0x13.0mm_Layout2x3x16_P0.8mm" (id 2) (at 248.92 151.13 0)
+    (property "Footprint" "footprints:BGA-96_9.0x13.0mm_P0.8mm" (id 2) (at 248.92 151.13 0)
       (effects (font (size 1.1938 1.1938)) hide)
     )
