File: pcb/mainboard/ec.kicad_sch (KiCad schematic)
At the start: 31 parts

Commit message: - pcb: r0p1 sch draft
Parts:
- gave numbers to parts that had none: 28
Connections:
- net +3V3 is gone; now on net +3V3_SB: C301.1, J301.1 (Pin_1), R303.1, U301.25 (USB1_VBUS), U301.27 (USB1_3V3), U301.61 (USB0_3V3)
- net EC_INT: now reaches U301.39 (PIO1_1)
- net PWR_EN: now reaches U301.41 (PIO1_2)
- net ARM_EN: now reaches U301.42 (PIO1_3)
Other:
- company: (none) -> Copyright EI-2030 2021.
- title: (none) -> Archer

Commit message: - pcb: start r0p1 layout
Parts:
- added U302: 74LS154, Package_SO:SO-24_5.3x15mm_P1.27mm, symbol 74xx:74LS154
- R301, R302, R303, R304: footprint Resistor_SMD:R_0603_1608Metric -> Resistor_SMD:R_0402_1005Metric
Connections:
- net +3V3_SB: now also U302.24 (VCC)
- net KSO0: now also U302.1 (S0); no longer U301.7 (PIO0_16)
- net KSO1: now also U302.2 (S1); no longer U301.3 (PIO0_17)
- net KSO10: now also U302.11 (S10); no longer U301.40 (PIO0_26)
- net KSO11: now also U302.13 (S11); no longer U301.18 (PIO0_27)
- net KSO12: now also U302.14 (S12); no longer U301.44 (PIO0_28)
- net KSO13: now also U302.15 (S13); no longer U301.59 (PIO0_29)
- net KSO14: now also U302.16 (S14); no longer U301.60 (PIO0_30)
- net KSO15: now also U302.17 (S15); no longer U301.15 (PIO0_31)
- net KSO2: now also U302.3 (S2); no longer U301.38 (PIO0_18)
- net KSO3: now also U302.4 (S3); no longer U301.58 (PIO0_19)
- net KSO4: now also U302.5 (S4); no longer U301.48 (PIO0_20)
- net KSO5: now also U302.6 (S5); no longer U301.49 (PIO0_21)
- net KSO6: now also U302.7 (S6); no longer U301.50 (PIO0_22)
- net KSO7: now also U302.8 (S7); no longer U301.12 (PIO0_23)
- net KSO8: now also U302.9 (S8); no longer U301.45 (PIO0_24)
- net KSO9: now also U302.10 (S9); no longer U301.51 (PIO0_25)
- net USB_OTG_ID: now reaches U301.4 (PIO1_0)
- new net: U302.12 (GND), U302.19 (E1)
- new net KSOE: U301.50 (PIO0_22), U302.18 (E0)
- new net KSOS1: U301.38 (PIO0_18), U302.23 (A0)
- new net KSOS2: U301.58 (PIO0_19), U302.22 (A1)
- new net KSOS3: U301.48 (PIO0_20), U302.21 (A2)
- new net KSOS4: U301.49 (PIO0_21), U302.20 (A3)
- new net LCD_EN: U301.44 (PIO0_28)
Other:
- company: Copyright EI-2030 2021. -> Copyright EI-2030 2021. / Engineer: Wenting Zhang
- title: Archer -> Archer Mainboard
- moved on the sheet: D301, J301, R303

Commit message: - pcb: components placed
Parts:
- removed D301: 1N5819, Diode_SMD:D_SOD-123, symbol Device:D_Schottky
- removed J301: Conn_02x05_Odd_Even, Connector_PinHeader_1.27mm:PinHeader_2x05_P1.27mm_Vertical_SMD, symbol Connector_Generic:Conn_02x05_Odd_Even
- removed R303: 10K, Resistor_SMD:R_0402_1005Metric, symbol Device:R
- added C317: 100nF, Capacitor_SMD:C_0402_1005Metric, symbol Device:C
- added J301: Conn_01x06_MountingPin, Connector_FFC-FPC:Hirose_FH12-6S-0.5SH_1x06-1MP_P0.50mm_Horizontal, symbol Connector_Generic_MountingPin:Conn_01x06_MountingPin
Connections:
- net +3V3_SB: now also C317.1, J301.1 (Pin_1)
- net GND: now also C317.2, J301.6 (Pin_6), J301.MP (MountPin)
- net UART1_TXD: now reaches U301.59 (PIO0_29)
- net UART1_RXD: now reaches U301.60 (PIO0_30)
- net DEBUG_USB_DP: now reaches U301.62 (USB0_DP)
- net DEBUG_USB_DM: now reaches U301.63 (USB0_DM)
- net MPU_JTAG_TCK renamed EC_SWCLK
- net EC_SWCLK: now also J301.4 (Pin_4)
- net MPU_JTAG_TMS renamed EC_SWDIO
- net EC_SWDIO: now also J301.5 (Pin_5)
- net POR renamed SB_PG
- no-connect marks 7 -> 4
Other:
- note removed: "ARM JTAG"
- moved on the sheet: C301

Commit message: - pcb: finishing layout r0p1
Connections:
- net GND: now also U302.12 (GND), U302.19 (E1)
- net KSO11: now also U302.17 (S15); no longer U302.13 (S11)
- net KSO12: now also U302.16 (S14); no longer U302.14 (S12)
- net KSO14: now also U302.14 (S12); no longer U302.16 (S14)
- net KSO15: now also U302.13 (S11); no longer U302.17 (S15)
- net SPI_LCD_CS: now reaches U301.12 (PIO0_23)
- net SPI_LCD_MISO: now reaches U301.40 (PIO0_26)
- net SPI_LCD_SCLK: now reaches U301.45 (PIO0_24)
- net SPI_LCD_MOSI: now reaches U301.51 (PIO0_25)
- net DEBUG_USB_DM renamed DEBUG_USB_D-
- net DEBUG_USB_DP renamed DEBUG_USB_D+
- net EC_SCL renamed EC_I2C_SCL
- net EC_SDA renamed EC_I2C_SDA
- net EC_USB_DM renamed EC_USB_D-
- net EC_USB_DP renamed EC_USB_D+
Changed lines of the file:
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@@
     (comment 4 "This source describes Open Hardware and is licensed under the CERN-OHL-S v2.")
   )
+  (junction (at 64.77 224.79) (diameter 0.9144) (color 0 0 0 0))
   (junction (at 76.2 78.74) (diameter 0.9144) (color 0 0 0 0))
   (junction (at 76.2 101.6) (diameter 0.9144) (color 0 0 0 0))
@@
     (stroke (width 0) (type solid) (color 0 0 0 0))
   )
+  (wire (pts (xy 53.34 127) (xy 58.42 127))
+    (stroke (width 0) (type solid) (color 0 0 0 0))
+  )
+  (wire (pts (xy 53.34 129.54) (xy 58.42 129.54))
+    (stroke (width 0) (type solid) (color 0 0 0 0))
+  )
+  (wire (pts (xy 53.34 132.08) (xy 58.42 132.08))
+    (stroke (width 0) (type solid) (color 0 0 0 0))
+  )
+  (wire (pts (xy 53.34 134.62) (xy 58.42 134.62))
+    (stroke (width 0) (type solid) (color 0 0 0 0))
+  )
   (wire (pts (xy 53.34 139.7) (xy 58.42 139.7))
     (stroke (width 0) (type solid) (color 0 0 0 0))
@@
     )
   )
+  (global_label "SPI_LCD_CS" (shape output) (at 58.42 127 0) (fields_autoplaced)
+    (effects (font (size 1.27 1.27)) (justify left))
+    (property "Intersheet References" "${INTERSHEET_REFS}" (id 0) (at 71.9002 126.9206 0)
+      (effects (font (size 1.27 1.27)) (justify left) hide)
+    )
+  )
+  (global_label "SPI_LCD_SCLK" (shape output) (at 58.42 129.54 0) (fields_autoplaced)
+    (effects (font (size 1.27 1.27)) (justify left))
+    (property "Intersheet References" "${INTERSHEET_REFS}" (id 0) (at 74.1983 129.4606 0)
+      (effects (font (size 1.27 1.27)) (justify left) hide)
+    )
+  )
+  (global_label "SPI_LCD_MOSI" (shape output) (at 58.42 132.08 0) (fields_autoplaced)
+    (effects (font (size 1.27 1.27)) (justify left))
+    (property "Intersheet References" "${INTERSHEET_REFS}" (id 0) (at 74.0169 132.0006 0)
+      (effects (font (size 1.27 1.27)) (justify left) hide)
+    )
+  )
+  (global_label "SPI_LCD_MISO" (shape output) (at 58.42 134.62 0) (fields_autoplaced)
+    (effects (font (size 1.27 1.27)) (justify left))
+    (property "Intersheet References" "${INTERSHEET_REFS}" (id 0) (at 74.0169 134.5406 0)
+      (effects (font (size 1.27 1.27)) (justify left) hide)
+    )
+  )
   (global_label "LCD_EN" (shape output) (at 58.42 139.7 0) (fields_autoplaced)
     (effects (font (size 1.27 1.27)) (justify left))
@@
     )
   )
-  (global_label "KSO11" (shape output) (at 80.01 207.01 0) (fields_autoplaced)
-    (effects (font (size 1.27 1.27)) (justify left))
-    (property "Intersheet References" "${INTERSHEET_REFS}" (id 0) (at 87.4426 206.9306 0)
-      (effects (font (size 1.27 1.27)) (justify left) hide)
-    )
-  )
-  (global_label "KSO12" (shape output) (at 80.01 209.55 0) (fields_autoplaced)
-    (effects (font (size 1.27 1.27)) (justify left))
-    (property "Intersheet References" "${INTERSHEET_REFS}" (id 0) (at 87.4426 209.4706 0)
+  (global_label "KSO15" (shape output) (at 80.01 207.01 0) (fields_autoplaced)
+    (effects (font (size 1.27 1.27)) (justify left))
+    (property "Intersheet References" "${INTERSHEET_REFS}" (id 0) (at 87.4426 207.0894 0)
+      (effects (font (size 1.27 1.27)) (justify left) hide)
+    )
+  )
+  (global_label "KSO14" (shape output) (at 80.01 209.55 0) (fields_autoplaced)
+    (effects (font (size 1.27 1.27)) (justify left))
+    (property "Intersheet References" "${INTERSHEET_REFS}" (id 0) (at 87.4426 209.6294 0)
       (effects (font (size 1.27 1.27)) (justify left) hide)
     )
@@
   (global_label "KSO13" (shape output) (at 80.01 212.09 0) (fields_autoplaced)
     (effects (font (size 1.27 1.27)) (justify left))
-    (property "Intersheet References" "${INTERSHEET_REFS}" (id 0) (at 87.4426 212.0106 0)
-      (effects (font (size 1.27 1.27)) (justify left) hide)
-    )
-  )
-  (global_label "KSO14" (shape output) (at 80.01 214.63 0) (fields_autoplaced)
-    (effects (font (size 1.27 1.27)) (justify left))
-    (property "Intersheet References" "${INTERSHEET_REFS}" (id 0) (at 87.4426 214.5506 0)
-      (effects (font (size 1.27 1.27)) (justify left) hide)
-    )
-  )
-  (global_label "KSO15" (shape output) (at 80.01 217.17 0) (fields_autoplaced)
-    (effects (font (size 1.27 1.27)) (justify left))
-    (property "Intersheet References" "${INTERSHEET_REFS}" (id 0) (at 87.4426 217.0906 0)
-      (effects (font (size 1.27 1.27)) (justify left) hide)
-    )
-  )
-  (global_label "EC_SDA" (shape bidirectional) (at 86.36 101.6 0) (fields_autoplaced)
-    (effects (font (size 1.27 1.27)) (justify left))
-    (property "Intersheet References" "${INTERSHEET_REFS}" (id 0) (at 95.7279 101.5206 0)
-      (effects (font (size 1.27 1.27)) (justify left) hide)
-    )
-  )
-  (global_label "EC_SCL" (shape output) (at 86.36 104.14 0) (fields_autoplaced)
-    (effects (font (size 1.27 1.27)) (justify left))
-    (property "Intersheet References" "${INTERSHEET_REFS}" (id 0) (at 95.6674 104.0606 0)
-      (effects (font (size 1.27 1.27)) (justify left) hide)
-    )
-  )
-  (global_label "DEBUG_USB_DP" (shape bidirectional) (at 140.97 49.53 180)
+    (property "Intersheet References" "${INTERSHEET_REFS}" (id 0) (at 87.4426 212.1694 0)
+      (effects (font (size 1.27 1.27)) (justify left) hide)
+    )
+  )
+  (global_label "KSO12" (shape output) (at 80.01 214.63 0) (fields_autoplaced)
+    (effects (font (size 1.27 1.27)) (justify left))
+    (property "Intersheet References" "${INTERSHEET_REFS}" (id 0) (at 87.4426 214.7094 0)
+      (effects (font (size 1.27 1.27)) (justify left) hide)
+    )
+  )
+  (global_label "KSO11" (shape output) (at 80.01 217.17 0) (fields_autoplaced)
+    (effects (font (size 1.27 1.27)) (justify left))
+    (property "Intersheet References" "${INTERSHEET_REFS}" (id 0) (at 87.4426 217.2494 0)
+      (effects (font (size 1.27 1.27)) (justify left) hide)
+    )
+  )
+  (global_label "EC_I2C_SDA" (shape bidirectional) (at 86.36 101.6 0) (fields_autoplaced)
+    (effects (font (size 1.27 1.27)) (justify left))
+    (property "Intersheet References" "${INTERSHEET_REFS}" (id 0) (at 99.7798 101.5206 0)
+      (effects (font (size 1.27 1.27)) (justify left) hide)
+    )
+  )
+  (global_label "EC_I2C_SCL" (shape output) (at 86.36 104.14 0) (fields_autoplaced)
+    (effects (font (size 1.27 1.27)) (justify left))
+    (property "Intersheet References" "${INTERSHEET_REFS}" (id 0) (at 99.7193 104.0606 0)
+      (effects (font (size 1.27 1.27)) (justify left) hide)
+    )
+  )
+  (global_label "DEBUG_USB_D+" (shape bidirectional) (at 140.97 49.53 180)
     (effects (font (size 1.27 1.27)) (justify right))
     (property "Intersheet References" "${INTERSHEET_REFS}" (id 0) (at 351.79 148.59 0)
@@
     )
   )
-  (global_label "DEBUG_USB_DM" (shape bidirectional) (at 140.97 52.07 180)
+  (global_label "DEBUG_USB_D-" (shape bidirectional) (at 140.97 52.07 180)
     (effects (font (size 1.27 1.27)) (justify right))
     (property "Intersheet References" "${INTERSHEET_REFS}" (id 0) (at 351.79 148.59 0)
@@
     )
   )
-  (global_label "EC_USB_DP" (shape bidirectional) (at 176.53 52.07 0)
+  (global_label "EC_USB_D+" (shape bidirectional) (at 176.53 52.07 0)
     (effects (font (size 1.27 1.27)) (justify left))
     (property "Intersheet References" "${INTERSHEET_REFS}" (id 0) (at -34.29 151.13 0)
@@
     )
   )
-  (global_label "EC_USB_DM" (shape bidirectional) (at 176.53 54.61 0)
+  (global_label "EC_USB_D-" (shape bidirectional) (at 176.53 54.61 0)
     (effects (font (size 1.27 1.27)) (justify left))
     (property "Intersheet References" "${INTERSHEET_REFS}" (id 0) (at -34.29 151.13 0)
@@
   (symbol (lib_id "symbols:+3V3_SB") (at 64.77 171.45 0) (unit 1)
     (in_bom yes) (on_board yes) (fields_autoplaced)
-    (property "Reference" "#PWR071" (id 0) (at 64.77 175.26 0)
+    (property "Reference" "#PWR0166" (id 0) (at 64.77 175.26 0)
       (effects (font (size 1.27 1.27)) hide)
     )
@@
       (effects (font (size 1.27 1.27)) hide)
     )
+    (pin "1")
+  )
+  (symbol (lib_id "power:GND") (at 64.77 224.79 0) (unit 1)
+    (in_bom yes) (on_board yes)
+    (property "Reference" "#PWR0163" (id 0) (at 64.77 231.14 0)
+      (effects (font (size 1.27 1.27)) hide)
+    )
+    (property "Value" "GND" (id 1) (at 68.58 226.06 0))
+    (property "Footprint" "" (id 2) (at 64.77 224.79 0)
+      (effects (font (size 1.27 1.27)) hide)
+    )
+    (property "Datasheet" "" (id 3) (at 64.77 224.79 0)
+      (effects (font (size 1.27 1.27)) hide)
+    )
