File: pcb/mainboard/power.kicad_sch (KiCad schematic)
At the start: 128 parts, among them J1 Conn_01x10_MountingPin, Q1 FDMC8327L, Q2 FDMC8327L, Q3 2SK3018, U1 SY8120, U101 MCIMX7S5EVM08SC, U2 SY8120, U3 SY8120, U4 SY8120, U5 SY8120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

Commit message: - pcb: finishing layout r0p1
Parts:
- added C82, C84: 10uF, Capacitor_SMD:C_0603_1608Metric, symbol Device:C
- added C83: 100nF, Capacitor_SMD:C_0402_1005Metric, symbol Device:C
- added U10: XC6206P122MR, Package_TO_SOT_SMD:SOT-23, symbol Regulator_Linear:XC6206PxxxMR
Connections:
- net 5V_EN is gone; now on net PWR_EN: U1.4 (RUN)
- net +1V8: now also C82.1, C83.1, U10.3 (VI)
- net GND: now also U101.J13 (VDDA_MIPI_1P8), U101.J15 (VDD_MIPI_1P0), U101.J17 (VDD_MIPI_1P0), C82.2, C83.2, C84.2, U10.1 (GND)
- net at C78.2, C79.2, C80.2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: no longer U101.J13 (VDDA_MIPI_1P8)
- net at C65.2, C76.2, C77.2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: no longer U101.J15 (VDD_MIPI_1P0), U101.J17 (VDD_MIPI_1P0)
- new net +1V2: C84.1, U10.2 (VO)
Other:
- moved on the sheet: C32, C33, C34, C36, C37, C38, C39, C40, C41, C42, C81, L7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

Commit message: - pcb: migrate to latest kicad, r0p1
Parts:
- added H1, H2, H3: MountingHole, MountingHole:MountingHole_2.2mm_M2_DIN965, symbol Mechanical:MountingHole
Changed lines of the file:
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@@
   (title_block
     (title "Archer Mainboard")
-    (date "2021-05-06")
-    (rev "R0.1 draft")
+    (date "2021-05-13")
+    (rev "R0.1")
     (company "Copyright EI-2030 2021. / Engineer: Wenting Zhang")
     (comment 2 "MERCHANTABILITY, SATISFACTORY QUALITY AND FITNESS FOR A PARTICULAR PURPOSE.")
@@
     (pin "2")
   )
+  (symbol (lib_id "Mechanical:MountingHole") (at 370.84 25.4 0) (unit 1)
+    (in_bom yes) (on_board yes) (fields_autoplaced)
+    (property "Reference" "H1" (id 0) (at 374.65 24.7649 0)
+      (effects (font (size 1.27 1.27)) (justify left))
+    )
+    (property "Value" "MountingHole" (id 1) (at 374.65 27.3049 0)
+      (effects (font (size 1.27 1.27)) (justify left))
+    )
+    (property "Footprint" "MountingHole:MountingHole_2.2mm_M2_DIN965" (id 2) (at 370.84 25.4 0)
+      (effects (font (size 1.27 1.27)) hide)
+    )
+    (property "Datasheet" "~" (id 3) (at 370.84 25.4 0)
+      (effects (font (size 1.27 1.27)) hide)
+    )
+  )
+  (symbol (lib_id "Mechanical:MountingHole") (at 370.84 33.02 0) (unit 1)
+    (in_bom yes) (on_board yes) (fields_autoplaced)
+    (property "Reference" "H2" (id 0) (at 374.65 32.3849 0)
+      (effects (font (size 1.27 1.27)) (justify left))
+    )
+    (property "Value" "MountingHole" (id 1) (at 374.65 34.9249 0)
+      (effects (font (size 1.27 1.27)) (justify left))
+    )
+    (property "Footprint" "MountingHole:MountingHole_2.2mm_M2_DIN965" (id 2) (at 370.84 33.02 0)
+      (effects (font (size 1.27 1.27)) hide)
+    )
+    (property "Datasheet" "~" (id 3) (at 370.84 33.02 0)
+      (effects (font (size 1.27 1.27)) hide)
+    )
+  )
+  (symbol (lib_id "Mechanical:MountingHole") (at 370.84 40.64 0) (unit 1)
+    (in_bom yes) (on_board yes) (fields_autoplaced)
+    (property "Reference" "H3" (id 0) (at 374.65 40.0049 0)
+      (effects (font (size 1.27 1.27)) (justify left))
+    )
+    (property "Value" "MountingHole" (id 1) (at 374.65 42.5449 0)
+      (effects (font (size 1.27 1.27)) (justify left))
+    )
+    (property "Footprint" "MountingHole:MountingHole_2.2mm_M2_DIN965" (id 2) (at 370.84 40.64 0)
+      (effects (font (size 1.27 1.27)) hide)
+    )
+    (property "Datasheet" "~" (id 3) (at 370.84 40.64 0)
+      (effects (font (size 1.27 1.27)) hide)
+    )
+  )
   (symbol (lib_id "Device:R") (at 111.76 57.15 180) (unit 1)
