File: pcb/mainboard/wifibt.kicad_sch (KiCad schematic)
At the start: 11 parts

Commit message: - pcb: working on r0p1 sch
Other:
- company: (none) -> Copyright EI-2030 2021.
- title: (none) -> Archer
Changed lines of the file:
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@@
 (kicad_sch (version 20210406) (generator eeschema)
   (paper "A4")
+  (title_block
+    (title "Archer")
+    (date "2021-04-26")
+    (rev "R0.1 draft")
+    (company "Copyright EI-2030 2021.")
+    (comment 2 "MERCHANTABILITY, SATISFACTORY QUALITY AND FITNESS FOR A PARTICULAR PURPOSE.")
+    (comment 3 "source is distributed WITHOUT ANY EXPRESS OR IMPLIED WARRANTY, INCLUDING OF")
+    (comment 4 "This source describes Open Hardware and is licensed under the CERN-OHL-S v2. This ")
+  )
   (junction (at 109.22 134.62) (diameter 0.9144) (color 0 0 0 0))
   (junction (at 121.92 134.62) (diameter 0.9144) (color 0 0 0 0))

Commit message: - pcb: r0p1 sch draft
Parts:
- gave numbers to parts that had none: 11
Changed lines of the file:
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@@
 (kicad_sch (version 20210406) (generator eeschema)
-  (paper "A4")
+  (paper "A3")
   (title_block
     (title "Archer")
@@
   (symbol (lib_id "power:+3V3") (at 175.26 66.04 0) (unit 1)
     (in_bom yes) (on_board yes)
-    (property "Reference" "#PWR?" (id 0) (at 175.26 69.85 0)
+    (property "Reference" "#PWR0906" (id 0) (at 175.26 69.85 0)
       (effects (font (size 1.27 1.27)) hide)
     )
@@
   (symbol (lib_id "power:GND") (at 99.06 139.7 0) (unit 1)
     (in_bom yes) (on_board yes)
-    (property "Reference" "#PWR?" (id 0) (at 99.06 146.05 0)
+    (property "Reference" "#PWR0901" (id 0) (at 99.06 146.05 0)
       (effects (font (size 1.27 1.27)) hide)
     )
@@
   (symbol (lib_id "power:GND") (at 109.22 147.32 0) (unit 1)
     (in_bom yes) (on_board yes)
-    (property "Reference" "#PWR?" (id 0) (at 109.22 153.67 0)
+    (property "Reference" "#PWR0902" (id 0) (at 109.22 153.67 0)
       (effects (font (size 1.27 1.27)) hide)
     )
@@
   (symbol (lib_id "power:GND") (at 121.92 147.32 0) (unit 1)
     (in_bom yes) (on_board yes)
-    (property "Reference" "#PWR?" (id 0) (at 121.92 153.67 0)
+    (property "Reference" "#PWR0903" (id 0) (at 121.92 153.67 0)
       (effects (font (size 1.27 1.27)) hide)
     )
@@
   (symbol (lib_id "power:GND") (at 134.62 139.7 0) (unit 1)
     (in_bom yes) (on_board yes)
-    (property "Reference" "#PWR?" (id 0) (at 134.62 146.05 0)
+    (property "Reference" "#PWR0904" (id 0) (at 134.62 146.05 0)
       (effects (font (size 1.27 1.27)) hide)
     )
@@
   (symbol (lib_id "power:GND") (at 170.18 96.52 0) (unit 1)
     (in_bom yes) (on_board yes)
-    (property "Reference" "#PWR?" (id 0) (at 170.18 102.87 0)
+    (property "Reference" "#PWR0905" (id 0) (at 170.18 102.87 0)
       (effects (font (size 1.27 1.27)) hide)
     )
@@
   (symbol (lib_id "power:GND") (at 175.26 91.44 0) (unit 1)
     (in_bom yes) (on_board yes)
-    (property "Reference" "#PWR?" (id 0) (at 175.26 97.79 0)
+    (property "Reference" "#PWR0907" (id 0) (at 175.26 97.79 0)
       (effects (font (size 1.27 1.27)) hide)
     )
@@
   (symbol (lib_id "power:GND") (at 200.66 91.44 0) (unit 1)
     (in_bom yes) (on_board yes)
-    (property "Reference" "#PWR?" (id 0) (at 200.66 97.79 0)
+    (property "Reference" "#PWR0908" (id 0) (at 200.66 97.79 0)
       (effects (font (size 1.27 1.27)) hide)
     )
@@
   (symbol (lib_id "Device:R") (at 115.57 134.62 270) (unit 1)
     (in_bom yes) (on_board yes)
-    (property "Reference" "R?" (id 0) (at 109.22 132.08 90)
+    (property "Reference" "R901" (id 0) (at 109.22 132.08 90)
       (effects (font (size 1.27 1.27)) (justify left))
     )
@@
   (symbol (lib_id "Device:R") (at 134.62 69.85 0) (unit 1)
     (in_bom yes) (on_board yes)
-    (property "Reference" "R?" (id 0) (at 136.398 68.6816 0)
+    (property "Reference" "R902" (id 0) (at 136.398 68.6816 0)
       (effects (font (size 1.27 1.27)) (justify left))
     )
@@
   (symbol (lib_id "Device:C") (at 109.22 140.97 180) (unit 1)
     (in_bom yes) (on_board yes)
-    (property "Reference" "C?" (id 0) (at 112.141 139.8016 0)
+    (property "Reference" "C901" (id 0) (at 112.141 139.8016 0)
       (effects (font (size 1.27 1.27)) (justify right))
     )
@@
   (symbol (lib_id "Device:C") (at 121.92 140.97 180) (unit 1)
     (in_bom yes) (on_board yes)
-    (property "Reference" "C?" (id 0) (at 124.841 139.8016 0)
+    (property "Reference" "C902" (id 0) (at 124.841 139.8016 0)
       (effects (font (size 1.27 1.27)) (justify right))
     )
@@
   (symbol (lib_id "Device:C") (at 128.27 134.62 270) (unit 1)
     (in_bom yes) (on_board yes)
-    (property "Reference" "C?" (id 0) (at 123.19 132.08 90))
+    (property "Reference" "C903" (id 0) (at 123.19 132.08 90))
     (property "Value" "33pF/50V/5%" (id 1) (at 133.35 132.08 90))
     (property "Footprint" "Capacitor_SMD:C_0402_1005Metric" (id 2) (at 124.46 135.5852 0)
@@
   (symbol (lib_id "Device:C") (at 175.26 85.09 0) (unit 1)
     (in_bom yes) (on_board yes)
-    (property "Reference" "C?" (id 0) (at 178.181 83.9216 0)
+    (property "Reference" "C904" (id 0) (at 178.181 83.9216 0)
       (effects (font (size 1.27 1.27)) (justify left))
     )
@@
   (symbol (lib_id "Device:C") (at 187.96 85.09 0) (unit 1)
     (in_bom yes) (on_board yes)
-    (property "Reference" "C?" (id 0) (at 190.881 83.9216 0)
+    (property "Reference" "C905" (id 0) (at 190.881 83.9216 0)
       (effects (font (size 1.27 1.27)) (justify left))
     )
@@
   (symbol (lib_id "Device:C") (at 200.66 85.09 0) (unit 1)
     (in_bom yes) (on_board yes)
-    (property "Reference" "C?" (id 0) (at 203.581 83.9216 0)
+    (property "Reference" "C906" (id 0) (at 203.581 83.9216 0)
       (effects (font (size 1.27 1.27)) (justify left))
     )
@@
   (symbol (lib_id "Device:C") (at 213.36 85.09 0) (unit 1)
     (in_bom yes) (on_board yes)
-    (property "Reference" "C?" (id 0) (at 216.281 83.9216 0)
+    (property "Reference" "C907" (id 0) (at 216.281 83.9216 0)
       (effects (font (size 1.27 1.27)) (justify left))
     )
@@
   (symbol (lib_id "symbols:WIFI_ANT_ESP8266") (at 91.44 137.16 0) (mirror y) (unit 1)
     (in_bom yes) (on_board yes)
-    (property "Reference" "ANT?" (id 0) (at 92.9132 124.7902 0)
+    (property "Reference" "ANT901" (id 0) (at 92.9132 124.7902 0)
       (effects (font (size 1.524 1.524)))
     )
@@
   (symbol (lib_id "symbols:RTL8723BS") (at 152.4 106.68 0) (unit 1)
     (in_bom yes) (on_board yes)
-    (property "Reference" "U?" (id 0) (at 152.4 68.9102 0)
+    (property "Reference" "U901" (id 0) (at 152.4 68.9102 0)
       (effects (font (size 1.524 1.524)))
     )

Commit message: - pcb: start r0p1 layout
Parts:
- R902: footprint Resistor_SMD:R_0603_1608Metric -> Resistor_SMD:R_0402_1005Metric
Other:
- company: Copyright EI-2030 2021. -> Copyright EI-2030 2021. / Engineer: Wenting Zhang
- title: Archer -> Archer Mainboard
Changed lines of the file:
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@@
   (paper "A3")
   (title_block
-    (title "Archer")
-    (date "2021-04-26")
+    (title "Archer Mainboard")
+    (date "2021-05-05")
     (rev "R0.1 draft")
-    (company "Copyright EI-2030 2021.")
+    (company "Copyright EI-2030 2021. / Engineer: Wenting Zhang")
     (comment 2 "MERCHANTABILITY, SATISFACTORY QUALITY AND FITNESS FOR A PARTICULAR PURPOSE.")
-    (comment 3 "source is distributed WITHOUT ANY EXPRESS OR IMPLIED WARRANTY, INCLUDING OF")
-    (comment 4 "This source describes Open Hardware and is licensed under the CERN-OHL-S v2. This ")
+    (comment 3 "This source is distributed WITHOUT ANY EXPRESS OR IMPLIED WARRANTY, INCLUDING OF")
+    (comment 4 "This source describes Open Hardware and is licensed under the CERN-OHL-S v2.")
   )
   (junction (at 109.22 134.62) (diameter 0.9144) (color 0 0 0 0))
@@
       (effects (font (size 1.27 1.27)) (justify left))
     )
-    (property "Footprint" "Resistor_SMD:R_0603_1608Metric" (id 2) (at 132.842 69.85 90)
-      (effects (font (size 1.27 1.27)) hide)
-    )
+    (property "Footprint" "Resistor_SMD:R_0402_1005Metric" (id 2) (at 132.842 69.85 90)
+      (effects (font (size 1.27 1.27)) hide)
+    )

Commit message: - pcb: finishing layout r0p1
Connections:
- net GND: no longer U901.41 (GND)
- new net UART3_CTS: U901.41 (UART_RTS)
Other:
- note added: "Headset profile is not supported. Use A2DP instead."
- note removed: "Due to I/O voltage constraint, headset profile would not be supported. Use A2DP instead."
Changed lines of the file:
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@@
+    (stroke (width 0) (type solid) (color 0 0 0 0))
+  )
+  (wire (pts (xy 124.46 109.22) (xy 137.16 109.22))
     (stroke (width 0) (type solid) (color 0 0 0 0))
   )
@@
     (stroke (width 0) (type solid) (color 0 0 0 0))
   )
-  (text "Due to I/O voltage constraint,\nheadset profile would not be supported.\nUse A2DP instead."
+  (text "Headset profile is not supported.\nUse A2DP instead."
     (at 92.71 105.41 0)
     (effects (font (size 1.27 1.27)) (justify left bottom))
@@
     )
   )
+  (global_label "UART3_CTS" (shape output) (at 124.46 109.22 180) (fields_autoplaced)
+    (effects (font (size 1.27 1.27)) (justify right))
+    (property "Intersheet References" "${INTERSHEET_REFS}" (id 0) (at 111.7659 109.1406 0)
+      (effects (font (size 1.27 1.27)) (justify right) hide)
+    )
+  )
